File: RPL_PCB/untitled.sch (EAGLE design)
At the start: 0 parts

Commit message: CPU schematic and pinout complete.  Working on adding IMU and Barom
Parts:
- added U$3: (no value), QFP50P2200X2200X160-144N:STM32F446ZET6
Changed lines of the file:
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@@
 <?xml version="1.0" encoding="utf-8"?>
 <!DOCTYPE eagle SYSTEM "eagle.dtd">
-<eagle version="9.2.2">
+<eagle version="9.2.0">
 <drawing>
 <settings>
@@
 </classes>
 <parts>
+<part name="U$3" library="QFP50P2200X2200X160-144N" deviceset="STM32F446ZET6" device=""/>
 </parts>
 <sheets>
@@
 </plain>
 <instances>
+<instance part="U$3" gate="G$1" x="-2232.66" y="-22.86" rot="R180"/>
 </instances>
 <busses>
